Commit message: color changes and some physical settings changed

File: src/igvc_description/urdf/base.xacro (robot description, xacro)
@@ -26,5 +26,5 @@
         </geometry>
         <material name="body_color">
-          <color rgba="0.2 0.2 0.25 1"/>
+          <color rgba="0.15 0.15 0.18 1"/>
         </material>
       </visual>
@@ -46,5 +46,5 @@
   <parent link="base_link"/>
   <child link="chassis_link"/>
-  <origin xyz="0 0 0.05"/>
+  <origin xyz="0 0 0.1"/>
 </joint>
   </xacro:macro>

File: src/igvc_description/urdf/sensors.xacro (robot description, xacro)
@@ -46,5 +46,5 @@
       <parent link="chassis_link"/>
       <child link="lidar_link"/>
-      <origin xyz="0.25 0 0.15"/>
+      <origin xyz="0 0 0.22"/>
     </joint>
     <!-- ================= DEPTH CAMERA ================= -->
@@ -73,5 +73,5 @@
       <parent link="chassis_link"/>
       <child link="camera_link"/>
-      <origin xyz="0.30 0 0.12"/>
+      <origin xyz="0.27 0 0.15"/>
     </joint>
   </xacro:macro>

File: src/igvc_description/urdf/wheels.xacro (robot description, xacro)
@@ -13,5 +13,5 @@
       </geometry>
       <material name="wheel_orange">
-        <color rgba="1.0 0.4 0.0 1"/>
+        <color rgba="1.0 0.25 0.0 1"/>
       </material>
     </visual>
