Commit message: physical changes to bot with sensors and wheels

File: install/igvc_description/share/igvc_description/urdf/base.xacro (robot description, xacro)
@@ -44,8 +44,8 @@
     <!-- Fixed joint connecting base_link to chassis -->
     <joint name="base_to_chassis" type="fixed">
-      <parent link="base_link"/>
-      <child link="chassis_link"/>
-      <origin xyz="0 0 0"/>
-    </joint>
+  <parent link="base_link"/>
+  <child link="chassis_link"/>
+  <origin xyz="0 0 0.05"/>
+</joint>
   </xacro:macro>
 </robot>

File: install/igvc_description/share/igvc_description/urdf/gazebo_plugins.xacro (robot description, xacro)
@@ -2,27 +2,15 @@
 <robot xmlns:xacro="http://www.ros.org/wiki/xacro">
   <xacro:macro name="gazebo_plugins">
-    <!-- IMU -->
+    <!-- IMU System -->
     <gazebo>
-      <plugin name="imu_plugin"
-              filename="libgz-sim-imu-system.so">
-        <topic>/imu/data</topic>
-        <frame_id>imu_link</frame_id>
-      </plugin>
+      <plugin
+        filename="libgz-sim-imu-system.so"
+        name="gz::sim::systems::Imu"/>
     </gazebo>
-    <!-- LIDAR -->
+    <!-- Sensors System (handles lidar + camera) -->
     <gazebo>
-      <plugin name="lidar_plugin"
-              filename="libgz-sim-lidar-system.so">
-        <topic>/scan</topic>
-        <frame_id>lidar_link</frame_id>
-      </plugin>
-    </gazebo>
-    <!-- Depth Camera -->
-    <gazebo>
-      <plugin name="camera_plugin"
-              filename="libgz-sim-depth-camera-system.so">
-        <camera_name>front_camera</camera_name>
-        <frame_id>camera_link</frame_id>
-      </plugin>
+      <plugin
+        filename="libgz-sim-sensors-system.so"
+        name="gz::sim::systems::Sensors"/>
     </gazebo>
   </xacro:macro>

File: install/igvc_description/share/igvc_description/urdf/sensors.xacro (robot description, xacro)
@@ -1,28 +1,60 @@
 <?xml version="1.0"?>
 <robot xmlns:xacro="http://www.ros.org/wiki/xacro">
-  <!-- Macro that adds all sensors -->
   <xacro:macro name="sensors">
     <!-- ================= IMU ================= -->
-    <link name="imu_link"/>
+    <link name="imu_link">
+      <sensor name="imu_sensor" type="imu">
+        <always_on>true</always_on>
+        <update_rate>100</update_rate>
+      </sensor>
+    </link>
     <joint name="imu_joint" type="fixed">
       <parent link="chassis_link"/>
       <child link="imu_link"/>
-      <!-- IMU placed on top of chassis -->
       <origin xyz="0 0 0.12"/>
     </joint>
-    <!-- ================= 2D LiDAR ================= -->
-    <link name="lidar_link"/>
+    <!-- ================= LIDAR ================= -->
+    <link name="lidar_link">
+      <sensor name="lidar_sensor" type="gpu_lidar">
+        <always_on>true</always_on>
+        <update_rate>10</update_rate>
+        <topic>/scan</topic>
+        <lidar>
+          <scan>
+            <horizontal>
+              <samples>720</samples>
+              <min_angle>-3.14159</min_angle>
+              <max_angle>3.14159</max_angle>
+            </horizontal>
+          </scan>
+          <range>
+            <min>0.12</min>
+            <max>10.0</max>
+          </range>
+        </lidar>
+      </sensor>
+    </link>
     <joint name="lidar_joint" type="fixed">
       <parent link="chassis_link"/>
       <child link="lidar_link"/>
-      <!-- LiDAR at front-top -->
       <origin xyz="0.25 0 0.15"/>
     </joint>
-    <!-- ================= RGB-D Camera ================= -->
-    <link name="camera_link"/>
+    <!-- ================= DEPTH CAMERA ================= -->
+    <link name="camera_link">
+      <sensor name="camera_sensor" type="depth_camera">
+        <always_on>true</always_on>
+        <update_rate>30</update_rate>
+        <camera>
+          <horizontal_fov>1.047</horizontal_fov>
+          <image>
+            <width>640</width>
+            <height>480</height>
+          </image>
+        </camera>
+      </sensor>
+    </link>
     <joint name="camera_joint" type="fixed">
       <parent link="chassis_link"/>
       <child link="camera_link"/>
-      <!-- Camera at front -->
       <origin xyz="0.30 0 0.12"/>
     </joint>

File: install/igvc_description/share/igvc_description/urdf/wheels.xacro (robot description, xacro)
@@ -40,8 +40,8 @@
     </joint>
   </xacro:macro>
-  <xacro:make_wheel name="wheel_fl" x="0.2"  y="0.18"  z="-0.1"/>
-  <xacro:make_wheel name="wheel_fr" x="0.2"  y="-0.18" z="-0.1"/>
-  <xacro:make_wheel name="wheel_rl" x="-0.2" y="0.18"  z="-0.1"/>
-  <xacro:make_wheel name="wheel_rr" x="-0.2" y="-0.18" z="-0.1"/>
+<xacro:make_wheel name="wheel_fl" x="0.2" y="0.18" z="-0.05"/>
+<xacro:make_wheel name="wheel_fr" x="0.2" y="-0.18" z="-0.05"/>
+<xacro:make_wheel name="wheel_rl" x="-0.2" y="0.18" z="-0.05"/>
+<xacro:make_wheel name="wheel_rr" x="-0.2" y="-0.18" z="-0.05"/>
 </xacro:macro>
 </robot>

File: src/igvc_description/urdf/base.xacro (robot description, xacro)
@@ -25,6 +25,6 @@
           <box size="0.5 0.4 0.2"/>
         </geometry>
-        <material name="grey">
-          <color rgba="0.6 0.6 0.6 1"/>
+        <material name="body_color">
+          <color rgba="0.2 0.2 0.25 1"/>
         </material>
       </visual>
@@ -44,8 +44,8 @@
     <!-- Fixed joint connecting base_link to chassis -->
     <joint name="base_to_chassis" type="fixed">
-      <parent link="base_link"/>
-      <child link="chassis_link"/>
-      <origin xyz="0 0 0"/>
-    </joint>
+  <parent link="base_link"/>
+  <child link="chassis_link"/>
+  <origin xyz="0 0 0.05"/>
+</joint>
   </xacro:macro>
 </robot>

File: src/igvc_description/urdf/sensors.xacro (robot description, xacro)
@@ -1,28 +1,78 @@
 <?xml version="1.0"?>
 <robot xmlns:xacro="http://www.ros.org/wiki/xacro">
-  <!-- Macro that adds all sensors -->
   <xacro:macro name="sensors">
     <!-- ================= IMU ================= -->
-    <link name="imu_link"/>
+    <link name="imu_link">
+      <sensor name="imu_sensor" type="imu">
+        <always_on>true</always_on>
+        <update_rate>100</update_rate>
+      </sensor>
+    </link>
     <joint name="imu_joint" type="fixed">
       <parent link="chassis_link"/>
       <child link="imu_link"/>
-      <!-- IMU placed on top of chassis -->
       <origin xyz="0 0 0.12"/>
     </joint>
-    <!-- ================= 2D LiDAR ================= -->
-    <link name="lidar_link"/>
+    <!-- ================= LIDAR ================= -->
+    <link name="lidar_link">
+  <visual>
+    <geometry>
+      <cylinder radius="0.04" length="0.05"/>
+    </geometry>
+    <material name="sensor_blue">
+      <color rgba="0.0 0.6 1.0 1"/>
+    </material>
+  </visual>
+</link>
+      <sensor name="lidar_sensor" type="gpu_lidar">
+        <always_on>true</always_on>
+        <update_rate>10</update_rate>
+        <topic>/scan</topic>
+        <lidar>
+          <scan>
+            <horizontal>
+              <samples>720</samples>
+              <min_angle>-3.14159</min_angle>
+              <max_angle>3.14159</max_angle>
+            </horizontal>
+          </scan>
+          <range>
+            <min>0.12</min>
+            <max>10.0</max>
+          </range>
+        </lidar>
+      </sensor>
+    </link>
     <joint name="lidar_joint" type="fixed">
       <parent link="chassis_link"/>
       <child link="lidar_link"/>
-      <!-- LiDAR at front-top -->
       <origin xyz="0.25 0 0.15"/>
     </joint>
-    <!-- ================= RGB-D Camera ================= -->
-    <link name="camera_link"/>
+    <!-- ================= DEPTH CAMERA ================= -->
+    <link name="camera_link">
+  <visual>
+    <geometry>
+      <box size="0.05 0.05 0.05"/>
+    </geometry>
+    <material name="sensor_green">
+      <color rgba="0.0 1.0 0.3 1"/>
+    </material>
+  </visual>
+</link>
+      <sensor name="camera_sensor" type="depth_camera">
+        <always_on>true</always_on>
+        <update_rate>30</update_rate>
+        <camera>
+          <horizontal_fov>1.047</horizontal_fov>
+          <image>
+            <width>640</width>
+            <height>480</height>
+          </image>
+        </camera>
+      </sensor>
+    </link>
     <joint name="camera_joint" type="fixed">
       <parent link="chassis_link"/>
       <child link="camera_link"/>
-      <!-- Camera at front -->
       <origin xyz="0.30 0 0.12"/>
     </joint>

File: src/igvc_description/urdf/wheels.xacro (robot description, xacro)
@@ -7,10 +7,13 @@
   <xacro:macro name="make_wheel" params="name x y z">
     <link name="${name}_link">
-      <visual>
-        <origin xyz="0 0 0" rpy="1.5708 0 0"/>
-        <geometry>
-          <cylinder radius="${wheel_radius}" length="${wheel_width}"/>
-        </geometry>
-      </visual>
+     <visual>
+      <origin xyz="0 0 0" rpy="1.5708 0 0"/>
+      <geometry>
+        <cylinder radius="${wheel_radius}" length="${wheel_width}"/>
+      </geometry>
+      <material name="wheel_orange">
+        <color rgba="1.0 0.4 0.0 1"/>
+      </material>
+    </visual>
       <collision>
         <origin xyz="0 0 0" rpy="1.5708 0 0"/>
@@ -40,8 +43,8 @@
     </joint>
   </xacro:macro>
-  <xacro:make_wheel name="wheel_fl" x="0.2"  y="0.18"  z="-0.1"/>
-  <xacro:make_wheel name="wheel_fr" x="0.2"  y="-0.18" z="-0.1"/>
-  <xacro:make_wheel name="wheel_rl" x="-0.2" y="0.18"  z="-0.1"/>
-  <xacro:make_wheel name="wheel_rr" x="-0.2" y="-0.18" z="-0.1"/>
+<xacro:make_wheel name="wheel_fl" x="0.2" y="0.23" z="-0.05"/>
+<xacro:make_wheel name="wheel_fr" x="0.2" y="-0.23" z="-0.05"/>
+<xacro:make_wheel name="wheel_rl" x="-0.2" y="0.23" z="-0.05"/>
+<xacro:make_wheel name="wheel_rr" x="-0.2" y="-0.23" z="-0.05"/>
 </xacro:macro>
 </robot>

Commit message: corrected sensor file

File: install/igvc_description/share/igvc_description/urdf/base.xacro (robot description, xacro)
@@ -25,6 +25,6 @@
           <box size="0.5 0.4 0.2"/>
         </geometry>
-        <material name="grey">
-          <color rgba="0.6 0.6 0.6 1"/>
+        <material name="body_color">
+          <color rgba="0.2 0.2 0.25 1"/>
         </material>
       </visual>

File: install/igvc_description/share/igvc_description/urdf/sensors.xacro (robot description, xacro)
@@ -16,4 +16,13 @@
     <!-- ================= LIDAR ================= -->
     <link name="lidar_link">
+  <visual>
+    <geometry>
+      <cylinder radius="0.04" length="0.05"/>
+    </geometry>
+    <material name="sensor_blue">
+      <color rgba="0.0 0.6 1.0 1"/>
+    </material>
+  </visual>
+</link>
       <sensor name="lidar_sensor" type="gpu_lidar">
         <always_on>true</always_on>
@@ -42,4 +51,13 @@
     <!-- ================= DEPTH CAMERA ================= -->
     <link name="camera_link">
+  <visual>
+    <geometry>
+      <box size="0.05 0.05 0.05"/>
+    </geometry>
+    <material name="sensor_green">
+      <color rgba="0.0 1.0 0.3 1"/>
+    </material>
+  </visual>
+</link>
       <sensor name="camera_sensor" type="depth_camera">
         <always_on>true</always_on>

File: install/igvc_description/share/igvc_description/urdf/wheels.xacro (robot description, xacro)
@@ -7,10 +7,13 @@
   <xacro:macro name="make_wheel" params="name x y z">
     <link name="${name}_link">
-      <visual>
-        <origin xyz="0 0 0" rpy="1.5708 0 0"/>
-        <geometry>
-          <cylinder radius="${wheel_radius}" length="${wheel_width}"/>
-        </geometry>
-      </visual>
+     <visual>
+      <origin xyz="0 0 0" rpy="1.5708 0 0"/>
+      <geometry>
+        <cylinder radius="${wheel_radius}" length="${wheel_width}"/>
+      </geometry>
+      <material name="wheel_orange">
+        <color rgba="1.0 0.4 0.0 1"/>
+      </material>
+    </visual>
       <collision>
         <origin xyz="0 0 0" rpy="1.5708 0 0"/>
@@ -40,8 +43,8 @@
     </joint>
   </xacro:macro>
-<xacro:make_wheel name="wheel_fl" x="0.2" y="0.18" z="-0.05"/>
-<xacro:make_wheel name="wheel_fr" x="0.2" y="-0.18" z="-0.05"/>
-<xacro:make_wheel name="wheel_rl" x="-0.2" y="0.18" z="-0.05"/>
-<xacro:make_wheel name="wheel_rr" x="-0.2" y="-0.18" z="-0.05"/>
+<xacro:make_wheel name="wheel_fl" x="0.2" y="0.23" z="-0.05"/>
+<xacro:make_wheel name="wheel_fr" x="0.2" y="-0.23" z="-0.05"/>
+<xacro:make_wheel name="wheel_rl" x="-0.2" y="0.23" z="-0.05"/>
+<xacro:make_wheel name="wheel_rr" x="-0.2" y="-0.23" z="-0.05"/>
 </xacro:macro>
 </robot>

File: src/igvc_description/urdf/sensors.xacro (robot description, xacro)
@@ -16,13 +16,12 @@
     <!-- ================= LIDAR ================= -->
     <link name="lidar_link">
-  <visual>
-    <geometry>
-      <cylinder radius="0.04" length="0.05"/>
-    </geometry>
-    <material name="sensor_blue">
-      <color rgba="0.0 0.6 1.0 1"/>
-    </material>
-  </visual>
-</link>
+      <visual>
+        <geometry>
+          <cylinder radius="0.04" length="0.05"/>
+        </geometry>
+        <material name="sensor_blue">
+          <color rgba="0.0 0.6 1.0 1"/>
+        </material>
+      </visual>
       <sensor name="lidar_sensor" type="gpu_lidar">
         <always_on>true</always_on>
@@ -51,13 +50,12 @@
     <!-- ================= DEPTH CAMERA ================= -->
     <link name="camera_link">
-  <visual>
-    <geometry>
-      <box size="0.05 0.05 0.05"/>
-    </geometry>
-    <material name="sensor_green">
-      <color rgba="0.0 1.0 0.3 1"/>
-    </material>
-  </visual>
-</link>
+      <visual>
+        <geometry>
+          <box size="0.05 0.05 0.05"/>
+        </geometry>
+        <material name="sensor_green">
+          <color rgba="0.0 1.0 0.3 1"/>
+        </material>
+      </visual>
       <sensor name="camera_sensor" type="depth_camera">
         <always_on>true</always_on>

Commit message: changes to structure

File: install/igvc_description/share/igvc_description/urdf/base.xacro (robot description, xacro)
@@ -26,5 +26,5 @@
         </geometry>
         <material name="body_color">
-          <color rgba="0.2 0.2 0.25 1"/>
+          <color rgba="0.15 0.15 0.18 1"/>
         </material>
       </visual>
@@ -43,8 +43,8 @@
     </link>
     <!-- Fixed joint connecting base_link to chassis -->
-    <joint name="base_to_chassis" type="fixed">
+<joint name="base_to_chassis" type="fixed">
   <parent link="base_link"/>
   <child link="chassis_link"/>
-  <origin xyz="0 0 0.05"/>
+  <origin xyz="0 0 0"/>
 </joint>
   </xacro:macro>

File: install/igvc_description/share/igvc_description/urdf/wheels.xacro (robot description, xacro)
@@ -8,14 +8,14 @@
     <link name="${name}_link">
      <visual>
-      <origin xyz="0 0 0" rpy="1.5708 0 0"/>
+      <origin xyz="0 0 0" rpy="0 1.5708 0"/>
       <geometry>
         <cylinder radius="${wheel_radius}" length="${wheel_width}"/>
       </geometry>
       <material name="wheel_orange">
-        <color rgba="1.0 0.4 0.0 1"/>
+        <color rgba="1.0 0.25 0.0 1"/>
       </material>
     </visual>
       <collision>
-        <origin xyz="0 0 0" rpy="1.5708 0 0"/>
+        <origin xyz="0 0 0" rpy="0 1.5708 0"/>
         <geometry>
           <cylinder radius="${wheel_radius}" length="${wheel_width}"/>
@@ -38,13 +38,13 @@
       <child link="${name}_link"/>
       <origin xyz="${x} ${y} ${z}"/>
-      <axis xyz="0 0 1"/>
+      <axis xyz="0 1 0"/>
       <limit effort="10.0" velocity="20.0"/>
       <dynamics damping="0.1" friction="0.0"/>
     </joint>
   </xacro:macro>
-<xacro:make_wheel name="wheel_fl" x="0.2" y="0.23" z="-0.05"/>
-<xacro:make_wheel name="wheel_fr" x="0.2" y="-0.23" z="-0.05"/>
-<xacro:make_wheel name="wheel_rl" x="-0.2" y="0.23" z="-0.05"/>
-<xacro:make_wheel name="wheel_rr" x="-0.2" y="-0.23" z="-0.05"/>
+<xacro:make_wheel name="wheel_fl" x="0.2" y="0.215" z="-0.15"/>
+<xacro:make_wheel name="wheel_fr" x="0.2" y="-0.215" z="-0.15"/>
+<xacro:make_wheel name="wheel_rl" x="-0.2" y="0.215" z="-0.15"/>
+<xacro:make_wheel name="wheel_rr" x="-0.2" y="-0.215" z="-0.15"/>
 </xacro:macro>
 </robot>

File: src/igvc_description/urdf/base.xacro (robot description, xacro)
@@ -1,51 +1,43 @@
 <?xml version="1.0"?>
 <robot xmlns:xacro="http://www.ros.org/wiki/xacro">
-  <!-- This macro creates the main body of the robot -->
-  <xacro:macro name="base">
-    <!-- Root link -->
-    <link name="base_link">
-      <inertial>
+<xacro:macro name="base">
+  <!-- BASE LINK (GROUND REFERENCE) -->
+  <link name="base_link">
+    <inertial>
+      <origin xyz="0 0 0"/>
+      <mass value="0.1"/>
+      <inertia ixx="0.0001" iyy="0.0001" izz="0.0001"
+               ixy="0.0" ixz="0.0" iyz="0.0"/>
+    </inertial>
+  </link>
+  <!-- CHASSIS -->
+  <link name="chassis_link">
+    <visual>
+      <origin xyz="0 0 0.15"/>
+      <geometry>
+        <box size="0.5 0.4 0.2"/>
+      </geometry>
+      <material name="body_color">
+        <color rgba="0.15 0.15 0.18 1"/>
+      </material>
+    </visual>
+    <collision>
+      <origin xyz="0 0 0.15"/>
+      <geometry>
+        <box size="0.5 0.4 0.2"/>
+      </geometry>
+    </collision>
+    <inertial>
+      <origin xyz="0 0 0.15"/>
+      <mass value="10.0"/>
+      <inertia ixx="0.2" iyy="0.2" izz="0.2"
+               ixy="0.0" ixz="0.0" iyz="0.0"/>
+    </inertial>
+  </link>
+  <joint name="base_to_chassis" type="fixed">
+    <parent link="base_link"/>
+    <child link="chassis_link"/>
     <origin xyz="0 0 0"/>
-    <mass value="0.1"/>
-    <inertia
-      ixx="0.0001"
-      iyy="0.0001"
-      izz="0.0001"
-      ixy="0.0"
-      ixz="0.0"
-      iyz="0.0"/>
-      </inertial>
-    </link>
-    <!-- Chassis: the main body -->
-    <link name="chassis_link">
-      <visual>
-        <origin xyz="0 0 0"/>
-        <geometry>
-          <!-- A simple box: length width height -->
-          <box size="0.5 0.4 0.2"/>
-        </geometry>
-        <material name="body_color">
-          <color rgba="0.15 0.15 0.18 1"/>
-        </material>
-      </visual>
-      <collision>
-        <origin xyz="0 0 0"/>
-        <geometry>
-          <box size="0.5 0.4 0.2"/>
-        </geometry>
-      </collision>
-      <inertial>
-        <mass value="10.0"/>
-        <origin xyz="0 0 0"/>
-        <inertia ixx="0.2" iyy="0.2" izz="0.2"
-                 ixy="0.0" ixz="0.0" iyz="0.0"/>
-      </inertial>
-    </link>
-    <!-- Fixed joint connecting base_link to chassis -->
-    <joint name="base_to_chassis" type="fixed">
-  <parent link="base_link"/>
-  <child link="chassis_link"/>
-  <origin xyz="0 0 0.1"/>
-</joint>
-  </xacro:macro>
+  </joint>
+</xacro:macro>
 </robot>

File: src/igvc_description/urdf/wheels.xacro (robot description, xacro)
@@ -8,5 +8,5 @@
     <link name="${name}_link">
      <visual>
-      <origin xyz="0 0 0" rpy="1.5708 0 0"/>
+      <origin xyz="0 0 0" rpy="0 1.5708 0"/>
       <geometry>
         <cylinder radius="${wheel_radius}" length="${wheel_width}"/>
@@ -17,5 +17,5 @@
     </visual>
       <collision>
-        <origin xyz="0 0 0" rpy="1.5708 0 0"/>
+        <origin xyz="0 0 0" rpy="0 1.5708 0"/>
         <geometry>
           <cylinder radius="${wheel_radius}" length="${wheel_width}"/>
@@ -38,13 +38,13 @@
       <child link="${name}_link"/>
       <origin xyz="${x} ${y} ${z}"/>
-      <axis xyz="0 0 1"/>
+      <axis xyz="0 1 0"/>
       <limit effort="10.0" velocity="20.0"/>
       <dynamics damping="0.1" friction="0.0"/>
     </joint>
   </xacro:macro>
-<xacro:make_wheel name="wheel_fl" x="0.2" y="0.23" z="-0.05"/>
-<xacro:make_wheel name="wheel_fr" x="0.2" y="-0.23" z="-0.05"/>
-<xacro:make_wheel name="wheel_rl" x="-0.2" y="0.23" z="-0.05"/>
-<xacro:make_wheel name="wheel_rr" x="-0.2" y="-0.23" z="-0.05"/>
+<xacro:make_wheel name="wheel_fl" x="0.2" y="0.215" z="0.05"/>
+<xacro:make_wheel name="wheel_fr" x="0.2" y="-0.215" z="0.05"/>
+<xacro:make_wheel name="wheel_rl" x="-0.2" y="0.215" z="0.05"/>
+<xacro:make_wheel name="wheel_rr" x="-0.2" y="-0.215" z="0.05"/>
 </xacro:macro>
 </robot>
