Commit message: structure changes

File: install/igvc_description/share/igvc_description/urdf/base.xacro (robot description, xacro)
@@ -1,51 +1,34 @@
 <?xml version="1.0"?>
 <robot xmlns:xacro="http://www.ros.org/wiki/xacro">
-  <!-- This macro creates the main body of the robot -->
-  <xacro:macro name="base">
-    <!-- Root link -->
-    <link name="base_link">
-      <inertial>
-    <origin xyz="0 0 0"/>
-    <mass value="0.1"/>
-    <inertia
-      ixx="0.0001"
-      iyy="0.0001"
-      izz="0.0001"
-      ixy="0.0"
-      ixz="0.0"
-      iyz="0.0"/>
-      </inertial>
-    </link>
-    <!-- Chassis: the main body -->
-    <link name="chassis_link">
-      <visual>
-        <origin xyz="0 0 0"/>
-        <geometry>
-          <!-- A simple box: length width height -->
-          <box size="0.5 0.4 0.2"/>
-        </geometry>
-        <material name="body_color">
-          <color rgba="0.15 0.15 0.18 1"/>
-        </material>
-      </visual>
-      <collision>
-        <origin xyz="0 0 0"/>
-        <geometry>
-          <box size="0.5 0.4 0.2"/>
-        </geometry>
-      </collision>
-      <inertial>
-        <mass value="10.0"/>
-        <origin xyz="0 0 0"/>
-        <inertia ixx="0.2" iyy="0.2" izz="0.2"
-                 ixy="0.0" ixz="0.0" iyz="0.0"/>
-      </inertial>
-    </link>
-    <!-- Fixed joint connecting base_link to chassis -->
-<joint name="base_to_chassis" type="fixed">
-  <parent link="base_link"/>
-  <child link="chassis_link"/>
-  <origin xyz="0 0 0"/>
-</joint>
-  </xacro:macro>
+<xacro:macro name="base">
+  <!-- Ground reference -->
+  <link name="base_link"/>
+  <!-- Chassis -->
+  <link name="chassis_link">
+    <visual>
+      <geometry>
+        <box size="0.5 0.4 0.2"/>
+      </geometry>
+      <material name="body_color">
+        <color rgba="0.15 0.15 0.18 1"/>
+      </material>
+    </visual>
+    <collision>
+      <geometry>
+        <box size="0.5 0.4 0.2"/>
+      </geometry>
+    </collision>
+    <inertial>
+      <mass value="10.0"/>
+      <inertia ixx="0.2" iyy="0.2" izz="0.2"
+               ixy="0.0" ixz="0.0" iyz="0.0"/>
+    </inertial>
+  </link>
+  <!-- Lift chassis above ground -->
+  <joint name="base_to_chassis" type="fixed">
+    <parent link="base_link"/>
+    <child link="chassis_link"/>
+    <origin xyz="0 0 0.15"/>
+  </joint>
+</xacro:macro>
 </robot>

File: install/igvc_description/share/igvc_description/urdf/wheels.xacro (robot description, xacro)
@@ -35,5 +35,5 @@
     </link>
     <joint name="${name}_joint" type="continuous">
-      <parent link="chassis_link"/>
+      <parent link="base_link"/>
       <child link="${name}_link"/>
       <origin xyz="${x} ${y} ${z}"/>
@@ -43,8 +43,8 @@
     </joint>
   </xacro:macro>
-<xacro:make_wheel name="wheel_fl" x="0.2" y="0.215" z="-0.15"/>
-<xacro:make_wheel name="wheel_fr" x="0.2" y="-0.215" z="-0.15"/>
-<xacro:make_wheel name="wheel_rl" x="-0.2" y="0.215" z="-0.15"/>
-<xacro:make_wheel name="wheel_rr" x="-0.2" y="-0.215" z="-0.15"/>
+<xacro:make_wheel name="wheel_fl" x="0.2" y="0.215" z="-0.05"/>
+<xacro:make_wheel name="wheel_fr" x="0.2" y="-0.215" z="-0.05"/>
+<xacro:make_wheel name="wheel_rl" x="-0.2" y="0.215" z="-0.05"/>
+<xacro:make_wheel name="wheel_rr" x="-0.2" y="-0.215" z="-0.05"/>
 </xacro:macro>
 </robot>

File: src/igvc_description/urdf/base.xacro (robot description, xacro)
@@ -2,17 +2,9 @@
 <robot xmlns:xacro="http://www.ros.org/wiki/xacro">
 <xacro:macro name="base">
-  <!-- BASE LINK (GROUND REFERENCE) -->
-  <link name="base_link">
-    <inertial>
-      <origin xyz="0 0 0"/>
-      <mass value="0.1"/>
-      <inertia ixx="0.0001" iyy="0.0001" izz="0.0001"
-               ixy="0.0" ixz="0.0" iyz="0.0"/>
-    </inertial>
-  </link>
-  <!-- CHASSIS -->
+  <!-- Ground reference -->
+  <link name="base_link"/>
+  <!-- Chassis -->
   <link name="chassis_link">
     <visual>
-      <origin xyz="0 0 0.15"/>
       <geometry>
         <box size="0.5 0.4 0.2"/>
@@ -23,5 +15,4 @@
     </visual>
     <collision>
-      <origin xyz="0 0 0.15"/>
       <geometry>
         <box size="0.5 0.4 0.2"/>
@@ -29,5 +20,4 @@
     </collision>
     <inertial>
-      <origin xyz="0 0 0.15"/>
       <mass value="10.0"/>
       <inertia ixx="0.2" iyy="0.2" izz="0.2"
@@ -35,8 +25,9 @@
     </inertial>
   </link>
+  <!-- Lift chassis above ground -->
   <joint name="base_to_chassis" type="fixed">
     <parent link="base_link"/>
     <child link="chassis_link"/>
-    <origin xyz="0 0 0"/>
+    <origin xyz="0 0 0.15"/>
   </joint>
 </xacro:macro>

File: src/igvc_description/urdf/wheels.xacro (robot description, xacro)
@@ -35,5 +35,5 @@
     </link>
     <joint name="${name}_joint" type="continuous">
-      <parent link="chassis_link"/>
+      <parent link="base_link"/>
       <child link="${name}_link"/>
       <origin xyz="${x} ${y} ${z}"/>
@@ -43,8 +43,8 @@
     </joint>
   </xacro:macro>
-<xacro:make_wheel name="wheel_fl" x="0.2" y="0.215" z="0.05"/>
-<xacro:make_wheel name="wheel_fr" x="0.2" y="-0.215" z="0.05"/>
-<xacro:make_wheel name="wheel_rl" x="-0.2" y="0.215" z="0.05"/>
-<xacro:make_wheel name="wheel_rr" x="-0.2" y="-0.215" z="0.05"/>
+<xacro:make_wheel name="wheel_fl" x="0.2" y="0.215" z="-0.05"/>
+<xacro:make_wheel name="wheel_fr" x="0.2" y="-0.215" z="-0.05"/>
+<xacro:make_wheel name="wheel_rl" x="-0.2" y="0.215" z="-0.05"/>
+<xacro:make_wheel name="wheel_rr" x="-0.2" y="-0.215" z="-0.05"/>
 </xacro:macro>
 </robot>

Commit message: changed the chassis link to fully base link

File: install/igvc_description/share/igvc_description/urdf/base.xacro (robot description, xacro)
@@ -2,7 +2,5 @@
 <robot xmlns:xacro="http://www.ros.org/wiki/xacro">
 <xacro:macro name="base">
-  <!-- Ground reference -->
   <link name="base_link"/>
-  <!-- Chassis -->
   <link name="chassis_link">
     <visual>
@@ -25,9 +23,9 @@
     </inertial>
   </link>
-  <!-- Lift chassis above ground -->
+  <!-- LIFT CHASSIS HALF HEIGHT -->
   <joint name="base_to_chassis" type="fixed">
     <parent link="base_link"/>
     <child link="chassis_link"/>
-    <origin xyz="0 0 0.15"/>
+    <origin xyz="0 0 0.1"/>
   </joint>
 </xacro:macro>

File: install/igvc_description/share/igvc_description/urdf/wheels.xacro (robot description, xacro)
@@ -43,8 +43,8 @@
     </joint>
   </xacro:macro>
-<xacro:make_wheel name="wheel_fl" x="0.2" y="0.215" z="-0.05"/>
-<xacro:make_wheel name="wheel_fr" x="0.2" y="-0.215" z="-0.05"/>
-<xacro:make_wheel name="wheel_rl" x="-0.2" y="0.215" z="-0.05"/>
-<xacro:make_wheel name="wheel_rr" x="-0.2" y="-0.215" z="-0.05"/>
+<xacro:make_wheel name="wheel_fl" x="0.2" y="0.25" z="0.05"/>
+<xacro:make_wheel name="wheel_fr" x="0.2" y="-0.25" z="0.05"/>
+<xacro:make_wheel name="wheel_rl" x="-0.2" y="0.25" z="0.05"/>
+<xacro:make_wheel name="wheel_rr" x="-0.2" y="-0.25" z="0.05"/>
 </xacro:macro>
 </robot>

File: src/igvc_description/urdf/base.xacro (robot description, xacro)
@@ -2,33 +2,27 @@
 <robot xmlns:xacro="http://www.ros.org/wiki/xacro">
 <xacro:macro name="base">
-  <!-- Ground reference -->
-  <link name="base_link"/>
-  <!-- Chassis -->
-  <link name="chassis_link">
-    <visual>
-      <geometry>
-        <box size="0.5 0.4 0.2"/>
-      </geometry>
-      <material name="body_color">
-        <color rgba="0.15 0.15 0.18 1"/>
-      </material>
-    </visual>
-    <collision>
-      <geometry>
-        <box size="0.5 0.4 0.2"/>
-      </geometry>
-    </collision>
-    <inertial>
-      <mass value="10.0"/>
-      <inertia ixx="0.2" iyy="0.2" izz="0.2"
-               ixy="0.0" ixz="0.0" iyz="0.0"/>
-    </inertial>
-  </link>
-  <!-- Lift chassis above ground -->
-  <joint name="base_to_chassis" type="fixed">
-    <parent link="base_link"/>
-    <child link="chassis_link"/>
-    <origin xyz="0 0 0.15"/>
-  </joint>
+<link name="base_link">
+<visual>
+  <geometry>
+    <box size="0.5 0.4 0.2"/>
+  </geometry>
+  <origin xyz="0 0 0.15"/>
+  <material name="body_color">
+    <color rgba="0.15 0.15 0.18 1"/>
+  </material>
+</visual>
+<collision>
+  <geometry>
+    <box size="0.5 0.4 0.2"/>
+  </geometry>
+  <origin xyz="0 0 0.15"/>
+</collision>
+<inertial>
+  <mass value="10.0"/>
+  <origin xyz="0 0 0.15"/>
+  <inertia ixx="0.2" iyy="0.2" izz="0.2"
+           ixy="0" ixz="0" iyz="0"/>
+</inertial>
+</link>
 </xacro:macro>
 </robot>

File: src/igvc_description/urdf/sensors.xacro (robot description, xacro)
@@ -1,78 +1,47 @@
 <?xml version="1.0"?>
 <robot xmlns:xacro="http://www.ros.org/wiki/xacro">
-  <xacro:macro name="sensors">
-    <!-- ================= IMU ================= -->
-    <link name="imu_link">
-      <sensor name="imu_sensor" type="imu">
-        <always_on>true</always_on>
-        <update_rate>100</update_rate>
-      </sensor>
-    </link>
-    <joint name="imu_joint" type="fixed">
-      <parent link="chassis_link"/>
-      <child link="imu_link"/>
-      <origin xyz="0 0 0.12"/>
-    </joint>
-    <!-- ================= LIDAR ================= -->
-    <link name="lidar_link">
-      <visual>
-        <geometry>
-          <cylinder radius="0.04" length="0.05"/>
-        </geometry>
-        <material name="sensor_blue">
-          <color rgba="0.0 0.6 1.0 1"/>
-        </material>
-      </visual>
-      <sensor name="lidar_sensor" type="gpu_lidar">
-        <always_on>true</always_on>
-        <update_rate>10</update_rate>
-        <topic>/scan</topic>
-        <lidar>
-          <scan>
-            <horizontal>
-              <samples>720</samples>
-              <min_angle>-3.14159</min_angle>
-              <max_angle>3.14159</max_angle>
-            </horizontal>
-          </scan>
-          <range>
-            <min>0.12</min>
-            <max>10.0</max>
-          </range>
-        </lidar>
-      </sensor>
-    </link>
-    <joint name="lidar_joint" type="fixed">
-      <parent link="chassis_link"/>
-      <child link="lidar_link"/>
-      <origin xyz="0 0 0.22"/>
-    </joint>
-    <!-- ================= DEPTH CAMERA ================= -->
-    <link name="camera_link">
-      <visual>
-        <geometry>
-          <box size="0.05 0.05 0.05"/>
-        </geometry>
-        <material name="sensor_green">
-          <color rgba="0.0 1.0 0.3 1"/>
-        </material>
-      </visual>
-      <sensor name="camera_sensor" type="depth_camera">
-        <always_on>true</always_on>
-        <update_rate>30</update_rate>
-        <camera>
-          <horizontal_fov>1.047</horizontal_fov>
-          <image>
-            <width>640</width>
-            <height>480</height>
-          </image>
-        </camera>
-      </sensor>
-    </link>
-    <joint name="camera_joint" type="fixed">
-      <parent link="chassis_link"/>
-      <child link="camera_link"/>
-      <origin xyz="0.27 0 0.15"/>
-    </joint>
-  </xacro:macro>
+<xacro:macro name="sensors">
+  <!-- ================= IMU ================= -->
+  <link name="imu_link"/>
+  <joint name="imu_joint" type="fixed">
+    <parent link="base_link"/>
+    <child link="imu_link"/>
+    <!-- slightly above top of body -->
+    <origin xyz="0 0 0.30"/>
+  </joint>
+  <!-- ================= LIDAR ================= -->
+  <link name="lidar_link">
+    <visual>
+      <geometry>
+        <cylinder radius="0.04" length="0.05"/>
+      </geometry>
+      <material name="sensor_blue">
+        <color rgba="0.0 0.6 1.0 1"/>
+      </material>
+    </visual>
+  </link>
+  <joint name="lidar_joint" type="fixed">
+    <parent link="base_link"/>
+    <child link="lidar_link"/>
+    <!-- front-top of robot -->
+    <origin xyz="0.15 0 0.30"/>
+  </joint>
+  <!-- ================= CAMERA ================= -->
+  <link name="camera_link">
+    <visual>
+      <geometry>
+        <box size="0.05 0.05 0.05"/>
+      </geometry>
+      <material name="sensor_green">
+        <color rgba="0.0 1.0 0.3 1"/>
+      </material>
+    </visual>
+  </link>
+  <joint name="camera_joint" type="fixed">
+    <parent link="base_link"/>
+    <child link="camera_link"/>
+    <!-- slightly forward -->
+    <origin xyz="0.22 0 0.27"/>
+  </joint>
+</xacro:macro>
 </robot>

File: src/igvc_description/urdf/wheels.xacro (robot description, xacro)
@@ -5,17 +5,17 @@
   <xacro:property name="wheel_width" value="0.03"/>
   <xacro:property name="wheel_mass" value="1.0"/>
-  <xacro:macro name="make_wheel" params="name x y z">
+  <xacro:macro name="make_wheel" params="name x y">
     <link name="${name}_link">
-     <visual>
-      <origin xyz="0 0 0" rpy="0 1.5708 0"/>
-      <geometry>
-        <cylinder radius="${wheel_radius}" length="${wheel_width}"/>
-      </geometry>
-      <material name="wheel_orange">
-        <color rgba="1.0 0.25 0.0 1"/>
-      </material>
-    </visual>
+      <visual>
+        <origin rpy="1.5708 0 0"/>
+        <geometry>
+          <cylinder radius="${wheel_radius}" length="${wheel_width}"/>
+        </geometry>
+        <material name="wheel_orange">
+          <color rgba="1.0 0.4 0.0 1"/>
+        </material>
+      </visual>
       <collision>
-        <origin xyz="0 0 0" rpy="0 1.5708 0"/>
+        <origin rpy="1.5708 0 0"/>
         <geometry>
           <cylinder radius="${wheel_radius}" length="${wheel_width}"/>
@@ -25,11 +25,6 @@
         <mass value="${wheel_mass}"/>
         <origin xyz="0 0 0"/>
-        <inertia
-          ixx="0.01"
-          iyy="0.01"
-          izz="0.01"
-          ixy="0.0"
-          ixz="0.0"
-          iyz="0.0"/>
+        <inertia ixx="0.01" iyy="0.01" izz="0.005"
+                 ixy="0.0" ixz="0.0" iyz="0.0"/>
       </inertial>
     </link>
@@ -37,14 +32,14 @@
       <parent link="base_link"/>
       <child link="${name}_link"/>
-      <origin xyz="${x} ${y} ${z}"/>
+      <!-- Wheel center at wheel_radius -->
+      <origin xyz="${x} ${y} ${wheel_radius}"/>
       <axis xyz="0 1 0"/>
-      <limit effort="10.0" velocity="20.0"/>
-      <dynamics damping="0.1" friction="0.0"/>
     </joint>
   </xacro:macro>
-<xacro:make_wheel name="wheel_fl" x="0.2" y="0.215" z="-0.05"/>
-<xacro:make_wheel name="wheel_fr" x="0.2" y="-0.215" z="-0.05"/>
-<xacro:make_wheel name="wheel_rl" x="-0.2" y="0.215" z="-0.05"/>
-<xacro:make_wheel name="wheel_rr" x="-0.2" y="-0.215" z="-0.05"/>
+  <!-- Slightly outside body width -->
+  <xacro:make_wheel name="wheel_fl" x="0.2"  y="0.25"/>
+  <xacro:make_wheel name="wheel_fr" x="0.2"  y="-0.25"/>
+  <xacro:make_wheel name="wheel_rl" x="-0.2" y="0.25"/>
+  <xacro:make_wheel name="wheel_rr" x="-0.2" y="-0.25"/>
 </xacro:macro>
 </robot>

Commit message: all structer sorted and keybindings done

File: install/igvc_description/share/igvc_description/urdf/base.xacro (robot description, xacro)
@@ -2,31 +2,27 @@
 <robot xmlns:xacro="http://www.ros.org/wiki/xacro">
 <xacro:macro name="base">
-  <link name="base_link"/>
-  <link name="chassis_link">
-    <visual>
-      <geometry>
-        <box size="0.5 0.4 0.2"/>
-      </geometry>
-      <material name="body_color">
-        <color rgba="0.15 0.15 0.18 1"/>
-      </material>
-    </visual>
-    <collision>
-      <geometry>
-        <box size="0.5 0.4 0.2"/>
-      </geometry>
-    </collision>
-    <inertial>
-      <mass value="10.0"/>
-      <inertia ixx="0.2" iyy="0.2" izz="0.2"
-               ixy="0.0" ixz="0.0" iyz="0.0"/>
-    </inertial>
-  </link>
-  <!-- LIFT CHASSIS HALF HEIGHT -->
-  <joint name="base_to_chassis" type="fixed">
-    <parent link="base_link"/>
-    <child link="chassis_link"/>
-    <origin xyz="0 0 0.1"/>
-  </joint>
+<link name="base_link">
+<visual>
+  <geometry>
+    <box size="0.5 0.4 0.2"/>
+  </geometry>
+  <origin xyz="0 0 0.15"/>
+  <material name="body_color">
+    <color rgba="0.15 0.15 0.18 1"/>
+  </material>
+</visual>
+<collision>
+  <geometry>
+    <box size="0.5 0.4 0.2"/>
+  </geometry>
+  <origin xyz="0 0 0.15"/>
+</collision>
+<inertial>
+  <mass value="10.0"/>
+  <origin xyz="0 0 0.15"/>
+  <inertia ixx="0.2" iyy="0.2" izz="0.2"
+           ixy="0" ixz="0" iyz="0"/>
+</inertial>
+</link>
 </xacro:macro>
 </robot>

File: install/igvc_description/share/igvc_description/urdf/wheels.xacro (robot description, xacro)
@@ -5,17 +5,17 @@
   <xacro:property name="wheel_width" value="0.03"/>
   <xacro:property name="wheel_mass" value="1.0"/>
-  <xacro:macro name="make_wheel" params="name x y z">
+  <xacro:macro name="make_wheel" params="name x y">
     <link name="${name}_link">
-     <visual>
-      <origin xyz="0 0 0" rpy="0 1.5708 0"/>
-      <geometry>
-        <cylinder radius="${wheel_radius}" length="${wheel_width}"/>
-      </geometry>
-      <material name="wheel_orange">
-        <color rgba="1.0 0.25 0.0 1"/>
-      </material>
-    </visual>
+      <visual>
+        <origin rpy="1.5708 0 0"/>
+        <geometry>
+          <cylinder radius="${wheel_radius}" length="${wheel_width}"/>
+        </geometry>
+        <material name="wheel_orange">
+          <color rgba="1.0 0.4 0.0 1"/>
+        </material>
+      </visual>
       <collision>
-        <origin xyz="0 0 0" rpy="0 1.5708 0"/>
+        <origin rpy="1.5708 0 0"/>
         <geometry>
           <cylinder radius="${wheel_radius}" length="${wheel_width}"/>
@@ -25,11 +25,6 @@
         <mass value="${wheel_mass}"/>
         <origin xyz="0 0 0"/>
-        <inertia
-          ixx="0.01"
-          iyy="0.01"
-          izz="0.01"
-          ixy="0.0"
-          ixz="0.0"
-          iyz="0.0"/>
+        <inertia ixx="0.01" iyy="0.01" izz="0.005"
+                 ixy="0.0" ixz="0.0" iyz="0.0"/>
       </inertial>
     </link>
@@ -37,14 +32,14 @@
       <parent link="base_link"/>
       <child link="${name}_link"/>
-      <origin xyz="${x} ${y} ${z}"/>
+      <!-- Wheel center at wheel_radius -->
+      <origin xyz="${x} ${y} ${wheel_radius}"/>
       <axis xyz="0 1 0"/>
-      <limit effort="10.0" velocity="20.0"/>
-      <dynamics damping="0.1" friction="0.0"/>
     </joint>
   </xacro:macro>
-<xacro:make_wheel name="wheel_fl" x="0.2" y="0.25" z="0.05"/>
-<xacro:make_wheel name="wheel_fr" x="0.2" y="-0.25" z="0.05"/>
-<xacro:make_wheel name="wheel_rl" x="-0.2" y="0.25" z="0.05"/>
-<xacro:make_wheel name="wheel_rr" x="-0.2" y="-0.25" z="0.05"/>
+  <!-- Slightly outside body width -->
+  <xacro:make_wheel name="wheel_fl" x="0.2"  y="0.21"/>
+  <xacro:make_wheel name="wheel_fr" x="0.2"  y="-0.21"/>
+  <xacro:make_wheel name="wheel_rl" x="-0.2" y="0.21"/>
+  <xacro:make_wheel name="wheel_rr" x="-0.2" y="-0.21"/>
 </xacro:macro>
 </robot>

File: src/igvc_description/urdf/wheels.xacro (robot description, xacro)
@@ -34,12 +34,12 @@
       <!-- Wheel center at wheel_radius -->
       <origin xyz="${x} ${y} ${wheel_radius}"/>
-      <axis xyz="0 1 0"/>
+      <axis xyz="0 0 1"/>
     </joint>
   </xacro:macro>
   <!-- Slightly outside body width -->
-  <xacro:make_wheel name="wheel_fl" x="0.2"  y="0.25"/>
-  <xacro:make_wheel name="wheel_fr" x="0.2"  y="-0.25"/>
-  <xacro:make_wheel name="wheel_rl" x="-0.2" y="0.25"/>
-  <xacro:make_wheel name="wheel_rr" x="-0.2" y="-0.25"/>
+  <xacro:make_wheel name="wheel_fl" x="0.2"  y="0.21"/>
+  <xacro:make_wheel name="wheel_fr" x="0.2"  y="-0.21"/>
+  <xacro:make_wheel name="wheel_rl" x="-0.2" y="0.21"/>
+  <xacro:make_wheel name="wheel_rr" x="-0.2" y="-0.21"/>
 </xacro:macro>
 </robot>

Commit message: changing sensors functionality to make them work

File: install/igvc_description/share/igvc_description/urdf/base.xacro (robot description, xacro)
@@ -3,26 +3,30 @@
 <xacro:macro name="base">
 <link name="base_link">
-<visual>
-  <geometry>
-    <box size="0.5 0.4 0.2"/>
-  </geometry>
-  <origin xyz="0 0 0.15"/>
-  <material name="body_color">
-    <color rgba="0.15 0.15 0.18 1"/>
-  </material>
-</visual>
-<collision>
-  <geometry>
-    <box size="0.5 0.4 0.2"/>
-  </geometry>
-  <origin xyz="0 0 0.15"/>
-</collision>
-<inertial>
-  <mass value="10.0"/>
-  <origin xyz="0 0 0.15"/>
-  <inertia ixx="0.2" iyy="0.2" izz="0.2"
-           ixy="0" ixz="0" iyz="0"/>
-</inertial>
+  <visual>
+    <geometry>
+      <box size="0.5 0.4 0.2"/>
+    </geometry>
+    <origin xyz="0 0 0.15"/>
+    <material name="body_color">
+      <color rgba="0.15 0.15 0.18 1"/>
+    </material>
+  </visual>
+  <collision>
+    <geometry>
+      <box size="0.5 0.4 0.2"/>
+    </geometry>
+    <origin xyz="0 0 0.15"/>
+  </collision>
+  <inertial>
+    <mass value="10.0"/>
+    <origin xyz="0 0 0.15"/>
+    <inertia ixx="0.2" iyy="0.2" izz="0.2"
+             ixy="0" ixz="0" iyz="0"/>
+  </inertial>
 </link>
+<!-- Correct gazebo tag placement -->
+<gazebo reference="base_link">
+  <self_collide>false</self_collide>
+</gazebo>
 </xacro:macro>
 </robot>

File: install/igvc_description/share/igvc_description/urdf/robot.xacro (robot description, xacro)
@@ -20,4 +20,5 @@
     <odom_frame>odom</odom_frame>
     <base_frame>base_link</base_frame>
+    <publish_tf>true</publish_tf>
     <left_joint>wheel_fl_joint</left_joint>
     <left_joint>wheel_rl_joint</left_joint>

File: install/igvc_description/share/igvc_description/urdf/sensors.xacro (robot description, xacro)
@@ -7,7 +7,13 @@
     <parent link="base_link"/>
     <child link="imu_link"/>
-    <!-- slightly above top of body -->
     <origin xyz="0 0 0.30"/>
   </joint>
+  <gazebo reference="imu_link">
+    <sensor name="imu_sensor" type="imu">
+      <always_on>true</always_on>
+      <update_rate>100</update_rate>
+      <topic>/imu</topic>
+    </sensor>
+  </gazebo>
   <!-- ================= LIDAR ================= -->
   <link name="lidar_link">
@@ -24,8 +30,29 @@
     <parent link="base_link"/>
     <child link="lidar_link"/>
-    <!-- front-top of robot -->
-    <origin xyz="0.15 0 0.30"/>
+    <origin xyz="0.15 0 0.55"/>
   </joint>
-  <!-- ================= CAMERA ================= -->
+  <gazebo reference="lidar_link">
+    <sensor name="lidar_link" type="gpu_lidar">
+      <always_on>true</always_on>
+      <update_rate>10</update_rate>
+      <topic>/scan</topic>
+      <frame_id>lidar_link</frame_id>
+      <visualize>true</visualize>
+<ray>
+  <scan>
+    <horizontal>
+      <samples>360</samples>
+      <min_angle>-3.14159</min_angle>
+      <max_angle>3.14159</max_angle>
+    </horizontal>
+  </scan>
+  <range>
+    <min>0.1</min>
+    <max>10.0</max>
+  </range>
+</ray>
+    </sensor>
+  </gazebo>
+  <!-- ================= CAMERA (visual only for now) -->
   <link name="camera_link">
     <visual>
@@ -41,5 +68,4 @@
     <parent link="base_link"/>
     <child link="camera_link"/>
-    <!-- slightly forward -->
     <origin xyz="0.22 0 0.27"/>
   </joint>
