Commit message: sensors

File: install/igvc_description/share/igvc_description/urdf/sensors.xacro (robot description, xacro)
@@ -22,8 +22,15 @@
         <cylinder radius="0.04" length="0.05"/>
       </geometry>
-      <material name="sensor_blue">
-        <color rgba="0.0 0.6 1.0 1"/>
-      </material>
     </visual>
+    <collision>
+      <geometry>
+        <cylinder radius="0.04" length="0.05"/>
+      </geometry>
+    </collision>
+    <inertial>
+      <mass value="0.1"/>
+      <inertia ixx="0.0001" iyy="0.0001" izz="0.0001"
+               ixy="0" ixz="0" iyz="0"/>
+    </inertial>
   </link>
   <joint name="lidar_joint" type="fixed">
@@ -32,27 +39,27 @@
     <origin xyz="0.15 0 0.55"/>
   </joint>
+  <!-- ✅ Stable CPU Ray Lidar (No GPU Crash) -->
   <gazebo reference="lidar_link">
-    <sensor name="lidar_link" type="gpu_lidar">
+    <sensor name="lidar" type="ray">
       <always_on>true</always_on>
       <update_rate>10</update_rate>
+      <visualize>true</visualize>
       <topic>/scan</topic>
-      <frame_id>lidar_link</frame_id>
-      <visualize>true</visualize>
-<ray>
-  <scan>
-    <horizontal>
-      <samples>360</samples>
-      <min_angle>-3.14159</min_angle>
-      <max_angle>3.14159</max_angle>
-    </horizontal>
-  </scan>
-  <range>
-    <min>0.1</min>
-    <max>10.0</max>
-  </range>
-</ray>
+      <ray>
+        <scan>
+          <horizontal>
+            <samples>360</samples>
+            <min_angle>-3.14159</min_angle>
+            <max_angle>3.14159</max_angle>
+          </horizontal>
+        </scan>
+        <range>
+          <min>0.1</min>
+          <max>10.0</max>
+        </range>
+      </ray>
     </sensor>
   </gazebo>
-  <!-- ================= CAMERA (visual only for now) -->
+  <!-- ================= CAMERA (visual only) ================= -->
   <link name="camera_link">
     <visual>

File: test.urdf (robot description, URDF)
Before this commit: robot igvc_bot, 9 links, 8 joints
Links:
- removed link chassis_link
- link base_link: mass None -> 10.0; geometry collision box size=0.5 0.4 0.2; visual box size=0.5 0.4 0.2
- link lidar_link: mass None -> 0.1; geometry collision cylinder length=0.05 radius=0.04; visual cylinder length=0.05 radius=0.04
Joints:
- removed joint base_to_chassis
- joint camera_joint: origin xyz=0.27 0 0.15 -> xyz=0.22 0 0.27; parent chassis_link -> base_link
- joint imu_joint: origin xyz=0 0 0.12 -> xyz=0 0 0.30; parent chassis_link -> base_link
- joint lidar_joint: origin xyz=0 0 0.22 -> xyz=0.15 0 0.55; parent chassis_link -> base_link
- joint wheel_fl_joint: limit effort=10.0 velocity=20.0 -> (none); origin xyz=0.2 0.215 -0.05 -> xyz=0.2 0.21 0.05
- joint wheel_fr_joint: limit effort=10.0 velocity=20.0 -> (none); origin xyz=0.2 -0.215 -0.05 -> xyz=0.2 -0.21 0.05
- joint wheel_rl_joint: limit effort=10.0 velocity=20.0 -> (none); origin xyz=-0.2 0.215 -0.05 -> xyz=-0.2 0.21 0.05
- joint wheel_rr_joint: limit effort=10.0 velocity=20.0 -> (none); origin xyz=-0.2 -0.215 -0.05 -> xyz=-0.2 -0.21 0.05
